File: PCB Design/GLEE_Testing_01_Advait.sch (EAGLE design)
At the start: 53 parts, among them IC1 SI7021, IC2 ATMEGA328-PB, IC3 PE4259, U1 V_REG_317SMD, U2 LSM9DS1, X1 LTI-SASF54GT, Y1 16MHz, Y2 32Mhz

Commit message: Final QA
Added a few changes, updated filenames, added library and BOM
Parts:
- removed C31: nc, SparkFun:CAP0402-CAP
- added C26: 100nF, SparkFun:CAP0402-CAP
- added R6: 220, SparkFun:RESISTOR0402-RES
- added R7: 360, SparkFun:RESISTOR0402-RES
- C1: value 26pF -> 10nF
- C10: value 10uF -> 1uF
- C11: value 10pF -> 47pF
- C12: value 0.1uF -> 1.2pF
- C13: value 10nF -> 33pF
- C14: value 0.1uF -> nc
- C15: value 100nF -> 4.7pF
- C16: value 47pF -> 1.8pF
- C18: value nc -> 1nF
- C19: value 33pF -> 47pF
- C2: value 26pF -> 0.1uF
- C20, L2: value 10nF -> nc
- C22: value 4.7pF -> 10nF
- C23: value 1.2pF -> nc
- C25: value 1.8pF -> 100nF
- C27: value 47pF -> 100nF
- C28: value 1nF -> 10pF
- C29: value nc -> 10pF
- C3: value 0.1 uF -> 0.1uF
- C4: value 1uF -> 10uF
- C6: value 10pF -> 0.1 uF
- C7, C9: value 100nF -> 26pF
- L1: value nc -> 10nH
- L3: value 10nH -> 6.2nH
- L4: value 6.2nH -> 0R
- L5: value 0R -> 10nF
- LED1: device adafruit:LED3MM -> adafruit:LEDCHIPLED_0805
- R1: value 10K -> 1K
- R3: value 220 -> 10K
- R4: value 360 -> 10K
- U1: value V_REG_317SMD -> LSM9DS1; device SparkFun:V_REG_317SMD -> LSM9DS1:LSM9DS1
- U2: value LSM9DS1 -> V_REG_317SMD; device LSM9DS1:LSM9DS1 -> SparkFun:V_REG_317SMD
Connections:
- new net N$56: R1.2, SW1.P$2
- net +3.3V: now also C18.1, C26.1, C6.1, R2.2, R3.1, R4.2, R5.1, R6.2, U1.SDO_A/G, U1.SDO_M, U1.VDD, U2.OUT; no longer C15.1, C28.1, C3.1, R1.1, R2.1, R3.2, R5.2, U1.OUT, U2.SDO_A/G, U2.SDO_M, U2.VDD
- net GND: now also C23.2, C24.2, C26.2, C27.2, R1.1, R7.1, U1.GND, U1.RES; no longer C11.2, C12.2, C13.2, C31.2, R4.1, SW1.P$2, U2.GND, U2.RES
- net I1: now also U1.DRDY_M; no longer U2.DRDY_M
- net I2: now also U1.INT2_A/G; no longer U2.INT2_A/G
- net I3: now also U1.INT_M; no longer U2.INT_M
- net I4: now also U1.INT1_A/G; no longer U2.INT1_A/G
- net N$1: now also C19.1; no longer C24.1
- net N$10: now also L5.2; no longer L2.2
- net N$11: now also C13.1, L2.1; no longer C19.1, L1.1
- net N$12: now also C12.1, C15.1, L1.2, L3.1; no longer C22.1, C23.1, L3.2, L4.1
- net N$13: now also C13.2, L1.1; no longer C19.2, L3.1
- net N$14: now also C12.2, C16.1, L3.2; no longer C23.2, C25.1, L4.2
- net N$15: now also C23.1, L4.2; no longer C31.1, L5.2
- net N$16: now also C11.1; no longer C27.1
- net N$17: now also C3.1, U1.C1; no longer C14.1, U2.C1
- net N$18: now also C11.2, C14.1, L4.1; no longer C27.2, C29.1, L5.1
- net N$2: now also C22.1, C24.1, L2.2; no longer C16.1, C20.1, L1.2
- net N$22: now also R4.1
- net N$24: now also C27.1; no longer C7.1
- net N$25: now also C25.1; no longer C9.1
- net N$3: now also U2.IN; no longer U1.IN
- net N$4: now also C19.2; no longer C24.2
- net N$5: now also R2.1, U1.CS_A/G, U1.CS_M; no longer R5.1, U2.CS_A/G, U2.CS_M
- net N$6: now also R6.1, R7.2, U2.ADJ; no longer R3.1, R4.2, U1.ADJ
- net N$7: now also C20.1, L5.1; no longer C18.1, L2.1
- net N$8: now also C1.1, U1.CAP; no longer C13.1, U2.CAP
- net N$9: now also C2.1, U1.VDDIO; no longer C12.1, U2.VDDIO
- net SCL: now also R3.2; no longer R1.2
- net SCL1: now also U1.SCL/SPC; no longer U2.SCL/SPC
- net SDA: now also R5.2; no longer R2.2
- net SDA1: now also U1.SDA/SDI/SDO; no longer U2.SDA/SDI/SDO
- net XTA: now also C28.1; no longer C6.1
- net XTAL1: now also C7.1; no longer C1.1
- net XTAL2: now also C9.1; no longer C2.1
- net XTB: now also C29.1; no longer C11.1
Other:
- moved on the sheet: C1, C10, C11, C12, C13, C14, C15, C16, C18, C19, C2, C20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

Commit message: Added pins for voltage testing
Parts:
- added JP6: (no value), pinhead:PINHD-1X2
- added R9: 100, SparkFun:RESISTOR0402-RES
Connections:
- new net N$19: LED1.A, R9.1
- net +3.3V: now also JP6.2, R9.2; no longer LED1.A
- net GND: now also JP6.1
Other:
- moved on the sheet: C7, C9, Y1
Changed lines of the file:
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@@
 <part name="R4" library="SparkFun" deviceset="RESISTOR" device="0402-RES" value="10K"/>
 <part name="R1" library="SparkFun" deviceset="RESISTOR" device="0402-RES" value="1K"/>
+<part name="JP6" library="pinhead" library_urn="urn:adsk.eagle:library:325" deviceset="PINHD-1X2" device="" package3d_urn="urn:adsk.eagle:package:22435/2"/>
+<part name="GND27" library="SparkFun" deviceset="GND" device=""/>
+<part name="R9" library="SparkFun" deviceset="RESISTOR" device="0402-RES" value="100"/>
 </parts>
 <sheets>
@@
 </instance>
 <instance part="IC2" gate="G$1" x="66.04" y="43.18" smashed="yes"/>
-<instance part="C9" gate="G$1" x="0" y="-5.08" smashed="yes">
-<attribute name="NAME" x="1.524" y="-2.159" size="1.778" layer="95"/>
-<attribute name="VALUE" x="1.524" y="-7.239" size="1.778" layer="96"/>
-</instance>
-<instance part="C7" gate="G$1" x="-20.32" y="-5.08" smashed="yes">
-<attribute name="NAME" x="-18.796" y="-2.159" size="1.778" layer="95"/>
-<attribute name="VALUE" x="-18.796" y="-7.239" size="1.778" layer="96"/>
-</instance>
-<instance part="GND22" gate="1" x="-10.16" y="-20.32" smashed="yes">
-<attribute name="VALUE" x="-12.7" y="-22.86" size="1.778" layer="96"/>
-</instance>
-<instance part="Y1" gate="G$1" x="-10.16" y="7.62" smashed="yes">
-<attribute name="NAME" x="-10.16" y="9.652" size="1.778" layer="95" font="vector" align="bottom-center"/>
-<attribute name="VALUE" x="-10.16" y="5.588" size="1.778" layer="96" font="vector" align="top-center"/>
+<instance part="C9" gate="G$1" x="0" y="-25.4" smashed="yes">
+<attribute name="NAME" x="1.524" y="-22.479" size="1.778" layer="95"/>
+<attribute name="VALUE" x="1.524" y="-27.559" size="1.778" layer="96"/>
+</instance>
+<instance part="C7" gate="G$1" x="-20.32" y="-25.4" smashed="yes">
+<attribute name="NAME" x="-18.796" y="-22.479" size="1.778" layer="95"/>
+<attribute name="VALUE" x="-18.796" y="-27.559" size="1.778" layer="96"/>
+</instance>
+<instance part="GND22" gate="1" x="-10.16" y="-40.64" smashed="yes">
+<attribute name="VALUE" x="-12.7" y="-43.18" size="1.778" layer="96"/>
+</instance>
+<instance part="Y1" gate="G$1" x="-10.16" y="-12.7" smashed="yes">
+<attribute name="NAME" x="-10.16" y="-10.668" size="1.778" layer="95" font="vector" align="bottom-center"/>
+<attribute name="VALUE" x="-10.16" y="-14.732" size="1.778" layer="96" font="vector" align="top-center"/>
 </instance>
 <instance part="R2" gate="G$1" x="241.3" y="124.46" smashed="yes">
@@
 <attribute name="NAME" x="128.0414" y="52.07" size="1.778" layer="95" rot="R90"/>
 <attribute name="VALUE" x="132.842" y="52.07" size="1.778" layer="96" rot="R90"/>
+</instance>
+<instance part="JP6" gate="G$1" x="116.84" y="134.62" smashed="yes" rot="R180">
+<attribute name="NAME" x="123.19" y="128.905" size="1.778" layer="95" rot="R180"/>
+<attribute name="VALUE" x="123.19" y="139.7" size="1.778" layer="96" rot="R180"/>
+</instance>
+<instance part="GND27" gate="1" x="127" y="124.46" smashed="yes">
+<attribute name="VALUE" x="124.46" y="121.92" size="1.778" layer="96"/>
+</instance>
+<instance part="R9" gate="G$1" x="124.46" y="106.68" smashed="yes" rot="R90">
+<attribute name="NAME" x="122.9614" y="102.87" size="1.778" layer="95" rot="R90"/>
+<attribute name="VALUE" x="127.762" y="102.87" size="1.778" layer="96" rot="R90"/>
 </instance>
 </instances>
@@
 </segment>
 <segment>
+<pinref part="IC1" gate="G$1" pin="GND@2"/>
 <pinref part="GND2" gate="1" pin="GND"/>
 <wire x1="-30.48" y1="33.02" x2="-30.48" y2="40.64" width="0.1524" layer="91"/>
-<pinref part="IC1" gate="G$1" pin="GND@2"/>
 <wire x1="-30.48" y1="40.64" x2="-25.4" y2="40.64" width="0.1524" layer="91"/>
 </segment>
@@
 <segment>
 <pinref part="C7" gate="G$1" pin="2"/>
-<wire x1="-20.32" y1="-7.62" x2="-20.32" y2="-12.7" width="0.1524" layer="91"/>
-<wire x1="-20.32" y1="-12.7" x2="-10.16" y2="-12.7" width="0.1524" layer="91"/>
+<wire x1="-20.32" y1="-27.94" x2="-20.32" y2="-33.02" width="0.1524" layer="91"/>
+<wire x1="-20.32" y1="-33.02" x2="-10.16" y2="-33.02" width="0.1524" layer="91"/>
 <pinref part="C9" gate="G$1" pin="2"/>
-<wire x1="-10.16" y1="-12.7" x2="0" y2="-12.7" width="0.1524" layer="91"/>
-<wire x1="0" y1="-12.7" x2="0" y2="-7.62" width="0.1524" layer="91"/>
-<wire x1="-10.16" y1="-12.7" x2="-10.16" y2="-17.78" width="0.1524" layer="91"/>
-<junction x="-10.16" y="-12.7"/>
+<wire x1="-10.16" y1="-33.02" x2="0" y2="-33.02" width="0.1524" layer="91"/>
+<wire x1="0" y1="-33.02" x2="0" y2="-27.94" width="0.1524" layer="91"/>
+<wire x1="-10.16" y1="-33.02" x2="-10.16" y2="-38.1" width="0.1524" layer="91"/>
+<junction x="-10.16" y="-33.02"/>
 <pinref part="GND22" gate="1" pin="GND"/>
 </segment>
@@
 <pinref part="GND35" gate="1" pin="GND"/>
 <wire x1="129.54" y1="50.8" x2="129.54" y2="48.26" width="0.1524" layer="91"/>
+</segment>
+<segment>
+<pinref part="JP6" gate="G$1" pin="1"/>
+<wire x1="119.38" y1="132.08" x2="127" y2="132.08" width="0.1524" layer="91"/>
+<wire x1="127" y1="132.08" x2="127" y2="127" width="0.1524" layer="91"/>
+<pinref part="GND27" gate="1" pin="GND"/>
 </segment>
 </net>
@@
 <wire x1="104.14" y1="121.92" x2="104.14" y2="124.46" width="0.1524" layer="91"/>
 <junction x="104.14" y="124.46"/>
-</segment>
-<segment>
-<pinref part="LED1" gate="G$1" pin="A"/>
-<wire x1="124.46" y1="96.52" x2="124.46" y2="101.6" width="0.1524" layer="91"/>
-<label x="124.46" y="101.6" size="1.778" layer="95" xref="yes"/>
+<wire x1="104.14" y1="124.46" x2="104.14" y2="134.62" width="0.1524" layer="91"/>
+<pinref part="JP6" gate="G$1" pin="2"/>
+<wire x1="104.14" y1="134.62" x2="119.38" y2="134.62" width="0.1524" layer="91"/>
+</segment>
+<segment>
+<label x="124.46" y="116.84" size="1.778" layer="95" xref="yes"/>
+<wire x1="124.46" y1="111.76" x2="124.46" y2="116.84" width="0.1524" layer="91"/>
+<pinref part="R9" gate="G$1" pin="2"/>
 </segment>
 <segment>
@@
 <segment>
 <pinref part="C7" gate="G$1" pin="1"/>
-<wire x1="-20.32" y1="0" x2="-20.32" y2="7.62" width="0.1524" layer="91"/>
-<label x="-20.32" y="12.7" size="1.778" layer="95" rot="R90" xref="yes"/>
+<wire x1="-20.32" y1="-20.32" x2="-20.32" y2="-12.7" width="0.1524" layer="91"/>
+<label x="-20.32" y="-7.62" size="1.778" layer="95" rot="R90" xref="yes"/>
 <pinref part="Y1" gate="G$1" pin="1"/>
-<wire x1="-20.32" y1="7.62" x2="-20.32" y2="12.7" width="0.1524" layer="91"/>
-<wire x1="-20.32" y1="7.62" x2="-12.7" y2="7.62" width="0.1524" layer="91"/>
-<junction x="-20.32" y="7.62"/>
+<wire x1="-20.32" y1="-12.7" x2="-20.32" y2="-7.62" width="0.1524" layer="91"/>
+<wire x1="-20.32" y1="-12.7" x2="-12.7" y2="-12.7" width="0.1524" layer="91"/>
+<junction x="-20.32" y="-12.7"/>
 </segment>
 <segment>
@@
 <segment>
 <pinref part="C9" gate="G$1" pin="1"/>
-<wire x1="0" y1="0" x2="0" y2="7.62" width="0.1524" layer="91"/>
-<label x="0" y="12.7" size="1.778" layer="95" rot="R90" xref="yes"/>
+<wire x1="0" y1="-20.32" x2="0" y2="-12.7" width="0.1524" layer="91"/>
+<label x="0" y="-7.62" size="1.778" layer="95" rot="R90" xref="yes"/>
 <pinref part="Y1" gate="G$1" pin="2"/>
-<wire x1="0" y1="7.62" x2="0" y2="12.7" width="0.1524" layer="91"/>
-<wire x1="-7.62" y1="7.62" x2="0" y2="7.62" width="0.1524" layer="91"/>
-<junction x="0" y="7.62"/>
+<wire x1="0" y1="-12.7" x2="0" y2="-7.62" width="0.1524" layer="91"/>
+<wire x1="-7.62" y1="-12.7" x2="0" y2="-12.7" width="0.1524" layer="91"/>
+<junction x="0" y="-12.7"/>
 </segment>
 </net>
@@
 </segment>
 </net>
+<net name="N$19" class="0">
+<segment>
+<pinref part="LED1" gate="G$1" pin="A"/>
+<wire x1="124.46" y1="96.52" x2="124.46" y2="101.6" width="0.1524" layer="91"/>
+<pinref part="R9" gate="G$1" pin="1"/>
+</segment>
+</net>
